Commit message: Add Gazebo simulation support and complete robot model
- Complete URDF with proper inertia, diff-drive wheels, caster, LiDAR, IMU
- Add Gazebo Harmonic plugins (diff-drive, joint state, GPU LiDAR, IMU)
- Add gazebo.launch.py with ros_gz_bridge for ROS2-Gazebo communication
- Add view_robot.launch.py for RViz visualization
- Add Ubuntu 24.04 setup script for native Linux development
- Add CLAUDE.md for Claude Code guidance

Co-Authored-By: Claude Opus 4.5 <noreply@anthropic.com>

File: ssbot_description/urdf/ssbot.urdf.xacro (robot description, xacro)
@@ -1,11 +1,111 @@
 <?xml version="1.0"?>
 <robot xmlns:xacro="http://www.ros.org/wiki/xacro" name="ssbot">
-  <!-- Properties -->
-  <xacro:property name="base_width" value="0.3"/>
-  <xacro:property name="base_length" value="0.4"/>
-  <xacro:property name="base_height" value="0.1"/>
-  <xacro:property name="wheel_radius" value="0.05"/>
-  <xacro:property name="wheel_width" value="0.03"/>
-  <!-- Base Link -->
+  <!-- ==================== Properties ==================== -->
+  <!-- Base dimensions (중형 로봇: 40cm x 35cm) -->
+  <xacro:property name="base_length" value="0.40"/>
+  <xacro:property name="base_width" value="0.35"/>
+  <xacro:property name="base_height" value="0.12"/>
+  <xacro:property name="base_mass" value="8.0"/>
+  <!-- Wheel properties -->
+  <xacro:property name="wheel_radius" value="0.065"/>
+  <xacro:property name="wheel_width" value="0.04"/>
+  <xacro:property name="wheel_mass" value="0.5"/>
+  <xacro:property name="wheel_separation" value="0.30"/>
+  <xacro:property name="wheel_offset_x" value="-0.05"/>
+  <!-- Caster properties -->
+  <xacro:property name="caster_radius" value="0.025"/>
+  <xacro:property name="caster_mass" value="0.1"/>
+  <xacro:property name="caster_offset_x" value="0.15"/>
+  <!-- LiDAR properties -->
+  <xacro:property name="lidar_radius" value="0.035"/>
+  <xacro:property name="lidar_height" value="0.045"/>
+  <xacro:property name="lidar_mass" value="0.2"/>
+  <xacro:property name="lidar_offset_z" value="0.08"/>
+  <!-- ==================== Materials ==================== -->
+  <material name="dark_gray">
+    <color rgba="0.3 0.3 0.3 1.0"/>
+  </material>
+  <material name="black">
+    <color rgba="0.1 0.1 0.1 1.0"/>
+  </material>
+  <material name="orange">
+    <color rgba="1.0 0.5 0.0 1.0"/>
+  </material>
+  <!-- ==================== Inertia Macros ==================== -->
+  <xacro:macro name="box_inertia" params="m x y z">
+    <inertial>
+      <mass value="${m}"/>
+      <inertia ixx="${m*(y*y+z*z)/12}" ixy="0" ixz="0"
+               iyy="${m*(x*x+z*z)/12}" iyz="0"
+               izz="${m*(x*x+y*y)/12}"/>
+    </inertial>
+  </xacro:macro>
+  <xacro:macro name="cylinder_inertia" params="m r h">
+    <inertial>
+      <mass value="${m}"/>
+      <inertia ixx="${m*(3*r*r+h*h)/12}" ixy="0" ixz="0"
+               iyy="${m*(3*r*r+h*h)/12}" iyz="0"
+               izz="${m*r*r/2}"/>
+    </inertial>
+  </xacro:macro>
+  <xacro:macro name="sphere_inertia" params="m r">
+    <inertial>
+      <mass value="${m}"/>
+      <inertia ixx="${2*m*r*r/5}" ixy="0" ixz="0"
+               iyy="${2*m*r*r/5}" iyz="0"
+               izz="${2*m*r*r/5}"/>
+    </inertial>
+  </xacro:macro>
+  <!-- ==================== Wheel Macro ==================== -->
+  <xacro:macro name="wheel" params="prefix side_reflect">
+    <link name="${prefix}_wheel_link">
+      <visual>
+        <geometry>
+          <cylinder radius="${wheel_radius}" length="${wheel_width}"/>
+        </geometry>
+        <origin xyz="0 0 0" rpy="${pi/2} 0 0"/>
+        <material name="black"/>
+      </visual>
+      <collision>
+        <geometry>
+          <cylinder radius="${wheel_radius}" length="${wheel_width}"/>
+        </geometry>
+        <origin xyz="0 0 0" rpy="${pi/2} 0 0"/>
+      </collision>
+      <xacro:cylinder_inertia m="${wheel_mass}" r="${wheel_radius}" h="${wheel_width}"/>
+    </link>
+    <joint name="${prefix}_wheel_joint" type="continuous">
+      <parent link="base_link"/>
+      <child link="${prefix}_wheel_link"/>
+      <origin xyz="${wheel_offset_x} ${side_reflect * wheel_separation/2} 0" rpy="0 0 0"/>
+      <axis xyz="0 1 0"/>
+      <dynamics damping="0.1" friction="0.1"/>
+    </joint>
+  </xacro:macro>
+  <!-- ==================== Caster Macro ==================== -->
+  <xacro:macro name="caster" params="prefix x_offset">
+    <link name="${prefix}_caster_link">
+      <visual>
+        <geometry>
+          <sphere radius="${caster_radius}"/>
+        </geometry>
+        <material name="dark_gray"/>
+      </visual>
+      <collision>
+        <geometry>
+          <sphere radius="${caster_radius}"/>
+        </geometry>
+      </collision>
+      <xacro:sphere_inertia m="${caster_mass}" r="${caster_radius}"/>
+    </link>
+    <joint name="${prefix}_caster_joint" type="fixed">
+      <parent link="base_link"/>
+      <child link="${prefix}_caster_link"/>
+      <origin xyz="${x_offset} 0 ${-base_height/2 - caster_radius + 0.005}" rpy="0 0 0"/>
+    </joint>
+  </xacro:macro>
+  <!-- ==================== Base Footprint ==================== -->
+  <link name="base_footprint"/>
+  <!-- ==================== Base Link ==================== -->
   <link name="base_link">
     <visual>
@@ -13,7 +113,5 @@
         <box size="${base_length} ${base_width} ${base_height}"/>
       </geometry>
-      <material name="blue">
-        <color rgba="0.0 0.0 0.8 1.0"/>
-      </material>
+      <material name="dark_gray"/>
     </visual>
     <collision>
@@ -22,11 +120,6 @@
       </geometry>
     </collision>
-    <inertial>
-      <mass value="5.0"/>
-      <inertia ixx="0.1" ixy="0" ixz="0" iyy="0.1" iyz="0" izz="0.1"/>
-    </inertial>
+    <xacro:box_inertia m="${base_mass}" x="${base_length}" y="${base_width}" z="${base_height}"/>
   </link>
-  <!-- Base Footprint (for navigation) -->
-  <link name="base_footprint"/>
   <joint name="base_footprint_joint" type="fixed">
     <parent link="base_footprint"/>
@@ -34,3 +127,46 @@
     <origin xyz="0 0 ${wheel_radius + base_height/2}" rpy="0 0 0"/>
   </joint>
+  <!-- ==================== Wheels ==================== -->
+  <xacro:wheel prefix="left" side_reflect="1"/>
+  <xacro:wheel prefix="right" side_reflect="-1"/>
+  <!-- ==================== Casters ==================== -->
+  <xacro:caster prefix="front" x_offset="${caster_offset_x}"/>
+  <!-- ==================== LiDAR ==================== -->
+  <link name="lidar_link">
+    <visual>
+      <geometry>
+        <cylinder radius="${lidar_radius}" length="${lidar_height}"/>
+      </geometry>
+      <origin xyz="0 0 0" rpy="0 0 0"/>
+      <material name="orange"/>
+    </visual>
+    <collision>
+      <geometry>
+        <cylinder radius="${lidar_radius}" length="${lidar_height}"/>
+      </geometry>
+      <origin xyz="0 0 0" rpy="0 0 0"/>
+    </collision>
+    <xacro:cylinder_inertia m="${lidar_mass}" r="${lidar_radius}" h="${lidar_height}"/>
+  </link>
+  <joint name="lidar_joint" type="fixed">
+    <parent link="base_link"/>
+    <child link="lidar_link"/>
+    <origin xyz="0 0 ${base_height/2 + lidar_offset_z}" rpy="0 0 0"/>
+  </joint>
+  <!-- LiDAR scan frame (센서 데이터 기준점) -->
+  <link name="laser_frame"/>
+  <joint name="laser_joint" type="fixed">
+    <parent link="lidar_link"/>
+    <child link="laser_frame"/>
+    <origin xyz="0 0 ${lidar_height/2}" rpy="0 0 0"/>
+  </joint>
+  <!-- ==================== IMU (Optional) ==================== -->
+  <link name="imu_link"/>
+  <joint name="imu_joint" type="fixed">
+    <parent link="base_link"/>
+    <child link="imu_link"/>
+    <origin xyz="0 0 0" rpy="0 0 0"/>
+  </joint>
+  <!-- ==================== Gazebo Plugins ==================== -->
+  <xacro:include filename="$(find ssbot_description)/urdf/gazebo.xacro"/>
 </robot>
