Commit message: Add dual LiDAR support and Cartographer SLAM
- Add ssbot_cartographer package for SLAM with dual NanoScan3 LiDARs
- Update gazebo.launch.py: remove headless-rendering for Native Ubuntu
- Add NanoScan3 driver launch and config files
- Add Gazebo world with sensor plugins
- Update robot model with front/rear LiDAR positions (1/7 o'clock)
- Configure ROS-Gazebo bridge for dual scan topics

Co-Authored-By: Claude Opus 4.5 <noreply@anthropic.com>

File: ssbot_description/urdf/gazebo.xacro (robot description, xacro)
@@ -15,11 +15,29 @@
     <mu2>1.0</mu2>
   </gazebo>
-  <gazebo reference="front_caster_link">
+  <gazebo reference="front_left_caster_link">
     <material>Gazebo/Grey</material>
     <mu1>0.0</mu1>
     <mu2>0.0</mu2>
   </gazebo>
-  <gazebo reference="lidar_link">
-    <material>Gazebo/Orange</material>
+  <gazebo reference="front_right_caster_link">
+    <material>Gazebo/Grey</material>
+    <mu1>0.0</mu1>
+    <mu2>0.0</mu2>
+  </gazebo>
+  <gazebo reference="rear_left_caster_link">
+    <material>Gazebo/Grey</material>
+    <mu1>0.0</mu1>
+    <mu2>0.0</mu2>
+  </gazebo>
+  <gazebo reference="rear_right_caster_link">
+    <material>Gazebo/Grey</material>
+    <mu1>0.0</mu1>
+    <mu2>0.0</mu2>
+  </gazebo>
+  <gazebo reference="front_lidar_link">
+    <material>Gazebo/Yellow</material>
+  </gazebo>
+  <gazebo reference="rear_lidar_link">
+    <material>Gazebo/Yellow</material>
   </gazebo>
   <!-- ==================== Differential Drive Plugin ==================== -->
@@ -28,6 +46,6 @@
       <left_joint>left_wheel_joint</left_joint>
       <right_joint>right_wheel_joint</right_joint>
-      <wheel_separation>0.30</wheel_separation>
-      <wheel_radius>0.065</wheel_radius>
+      <wheel_separation>0.35</wheel_separation>
+      <wheel_radius>0.08</wheel_radius>
       <odom_publish_frequency>50</odom_publish_frequency>
       <topic>cmd_vel</topic>
@@ -44,32 +62,63 @@
     </plugin>
   </gazebo>
-  <!-- ==================== 2D LiDAR Sensor ==================== -->
-  <gazebo reference="lidar_link">
-    <sensor name="lidar" type="gpu_lidar">
+  <!-- ==================== Front NanoScan3 LiDAR (1 o'clock) ==================== -->
+  <!-- SICK NanoScan3: 275° FOV, up to 3m safety / 40m detection -->
+  <gazebo reference="front_lidar_link">
+    <sensor name="front_lidar" type="gpu_lidar">
       <always_on>true</always_on>
-      <update_rate>10</update_rate>
+      <update_rate>15</update_rate>
       <visualize>true</visualize>
-      <topic>scan</topic>
+      <topic>scan_front</topic>
       <lidar>
         <scan>
           <horizontal>
-            <samples>360</samples>
+            <samples>275</samples>
             <resolution>1</resolution>
-            <min_angle>-3.14159</min_angle>
-            <max_angle>3.14159</max_angle>
+            <min_angle>-2.4</min_angle>
+            <max_angle>2.4</max_angle>
           </horizontal>
         </scan>
         <range>
-          <min>0.12</min>
-          <max>12.0</max>
-          <resolution>0.01</resolution>
+          <min>0.05</min>
+          <max>40.0</max>
+          <resolution>0.001</resolution>
         </range>
         <noise>
           <type>gaussian</type>
           <mean>0.0</mean>
-          <stddev>0.01</stddev>
+          <stddev>0.005</stddev>
         </noise>
       </lidar>
-      <frame_id>laser_frame</frame_id>
+      <frame_id>front_laser_frame</frame_id>
+    </sensor>
+  </gazebo>
+  <!-- ==================== Rear NanoScan3 LiDAR (7 o'clock) ==================== -->
+  <gazebo reference="rear_lidar_link">
+    <sensor name="rear_lidar" type="gpu_lidar">
+      <always_on>true</always_on>
+      <update_rate>15</update_rate>
+      <visualize>true</visualize>
+      <topic>scan_rear</topic>
+      <lidar>
+        <scan>
+          <horizontal>
+            <samples>275</samples>
+            <resolution>1</resolution>
+            <min_angle>-2.4</min_angle>
+            <max_angle>2.4</max_angle>
+          </horizontal>
+        </scan>
+        <range>
+          <min>0.05</min>
+          <max>40.0</max>
+          <resolution>0.001</resolution>
+        </range>
+        <noise>
+          <type>gaussian</type>
+          <mean>0.0</mean>
+          <stddev>0.005</stddev>
+        </noise>
+      </lidar>
+      <frame_id>rear_laser_frame</frame_id>
     </sensor>
   </gazebo>

File: ssbot_description/urdf/ssbot.urdf.xacro (robot description, xacro)
@@ -2,24 +2,38 @@
 <robot xmlns:xacro="http://www.ros.org/wiki/xacro" name="ssbot">
   <!-- ==================== Properties ==================== -->
-  <!-- Base dimensions (중형 로봇: 40cm x 35cm) -->
-  <xacro:property name="base_length" value="0.40"/>
-  <xacro:property name="base_width" value="0.35"/>
-  <xacro:property name="base_height" value="0.12"/>
-  <xacro:property name="base_mass" value="8.0"/>
+  <!-- Base dimensions: 600mm x 400mm -->
+  <xacro:property name="base_length" value="0.60"/>
+  <xacro:property name="base_width" value="0.40"/>
+  <xacro:property name="base_height" value="0.15"/>
+  <xacro:property name="base_mass" value="15.0"/>
   <!-- Wheel properties -->
-  <xacro:property name="wheel_radius" value="0.065"/>
-  <xacro:property name="wheel_width" value="0.04"/>
-  <xacro:property name="wheel_mass" value="0.5"/>
-  <xacro:property name="wheel_separation" value="0.30"/>
-  <xacro:property name="wheel_offset_x" value="-0.05"/>
-  <!-- Caster properties -->
-  <xacro:property name="caster_radius" value="0.025"/>
-  <xacro:property name="caster_mass" value="0.1"/>
-  <xacro:property name="caster_offset_x" value="0.15"/>
-  <!-- LiDAR properties -->
-  <xacro:property name="lidar_radius" value="0.035"/>
-  <xacro:property name="lidar_height" value="0.045"/>
-  <xacro:property name="lidar_mass" value="0.2"/>
-  <xacro:property name="lidar_offset_z" value="0.08"/>
+  <xacro:property name="wheel_radius" value="0.08"/>
+  <xacro:property name="wheel_width" value="0.05"/>
+  <xacro:property name="wheel_mass" value="0.8"/>
+  <xacro:property name="wheel_separation" value="0.35"/>
+  <xacro:property name="wheel_offset_x" value="0.0"/>
+  <xacro:property name="wheel_offset_z" value="${-base_height/2}"/>
+  <!-- Caster properties (4 corners) -->
+  <xacro:property name="caster_radius" value="0.03"/>
+  <xacro:property name="caster_mass" value="0.2"/>
+  <xacro:property name="caster_offset_x" value="0.25"/>
+  <xacro:property name="caster_offset_y" value="0.15"/>
+  <!-- Caster z: caster center should be at caster_radius from ground -->
+  <xacro:property name="caster_offset_z" value="${caster_radius - wheel_radius - base_height/2}"/>
+  <!-- SICK NanoScan3 properties -->
+  <!-- Dimensions: 80mm x 80mm x 101mm -->
+  <xacro:property name="lidar_size_x" value="0.08"/>
+  <xacro:property name="lidar_size_y" value="0.08"/>
+  <xacro:property name="lidar_size_z" value="0.101"/>
+  <xacro:property name="lidar_mass" value="0.5"/>
+  <!-- LiDAR positions (1 o'clock and 7 o'clock) -->
+  <!-- 1 o'clock: front-right corner -->
+  <xacro:property name="lidar_front_x" value="0.22"/>
+  <xacro:property name="lidar_front_y" value="-0.12"/>
+  <xacro:property name="lidar_front_yaw" value="${-pi/6}"/>
+  <!-- 7 o'clock: rear-left corner -->
+  <xacro:property name="lidar_rear_x" value="-0.22"/>
+  <xacro:property name="lidar_rear_y" value="0.12"/>
+  <xacro:property name="lidar_rear_yaw" value="${5*pi/6}"/>
   <!-- ==================== Materials ==================== -->
   <material name="dark_gray">
@@ -29,6 +43,6 @@
     <color rgba="0.1 0.1 0.1 1.0"/>
   </material>
-  <material name="orange">
-    <color rgba="1.0 0.5 0.0 1.0"/>
+  <material name="sick_yellow">
+    <color rgba="1.0 0.85 0.0 1.0"/>
   </material>
   <!-- ==================== Inertia Macros ==================== -->
@@ -78,5 +92,5 @@
       <parent link="base_link"/>
       <child link="${prefix}_wheel_link"/>
-      <origin xyz="${wheel_offset_x} ${side_reflect * wheel_separation/2} 0" rpy="0 0 0"/>
+      <origin xyz="${wheel_offset_x} ${side_reflect * wheel_separation/2} ${wheel_offset_z}" rpy="0 0 0"/>
       <axis xyz="0 1 0"/>
       <dynamics damping="0.1" friction="0.1"/>
@@ -84,5 +98,5 @@
   </xacro:macro>
   <!-- ==================== Caster Macro ==================== -->
-  <xacro:macro name="caster" params="prefix x_offset">
+  <xacro:macro name="caster" params="prefix x_reflect y_reflect">
     <link name="${prefix}_caster_link">
       <visual>
@@ -102,5 +116,36 @@
       <parent link="base_link"/>
       <child link="${prefix}_caster_link"/>
-      <origin xyz="${x_offset} 0 ${-base_height/2 - caster_radius + 0.005}" rpy="0 0 0"/>
+      <origin xyz="${x_reflect * caster_offset_x} ${y_reflect * caster_offset_y} ${caster_offset_z}" rpy="0 0 0"/>
+    </joint>
+  </xacro:macro>
+  <!-- ==================== NanoScan3 LiDAR Macro ==================== -->
+  <xacro:macro name="nanoscan3" params="prefix x y yaw topic">
+    <link name="${prefix}_lidar_link">
+      <visual>
+        <geometry>
+          <box size="${lidar_size_x} ${lidar_size_y} ${lidar_size_z}"/>
+        </geometry>
+        <origin xyz="0 0 0" rpy="0 0 0"/>
+        <material name="sick_yellow"/>
+      </visual>
+      <collision>
+        <geometry>
+          <box size="${lidar_size_x} ${lidar_size_y} ${lidar_size_z}"/>
+        </geometry>
+        <origin xyz="0 0 0" rpy="0 0 0"/>
+      </collision>
+      <xacro:box_inertia m="${lidar_mass}" x="${lidar_size_x}" y="${lidar_size_y}" z="${lidar_size_z}"/>
+    </link>
+    <joint name="${prefix}_lidar_joint" type="fixed">
+      <parent link="base_link"/>
+      <child link="${prefix}_lidar_link"/>
+      <origin xyz="${x} ${y} ${base_height/2 + lidar_size_z/2}" rpy="0 0 ${yaw}"/>
+    </joint>
+    <!-- Scan frame at the top of the LiDAR -->
+    <link name="${prefix}_laser_frame"/>
+    <joint name="${prefix}_laser_joint" type="fixed">
+      <parent link="${prefix}_lidar_link"/>
+      <child link="${prefix}_laser_frame"/>
+      <origin xyz="0 0 ${lidar_size_z/2}" rpy="0 0 0"/>
     </joint>
   </xacro:macro>
@@ -130,36 +175,23 @@
   <xacro:wheel prefix="left" side_reflect="1"/>
   <xacro:wheel prefix="right" side_reflect="-1"/>
-  <!-- ==================== Casters ==================== -->
-  <xacro:caster prefix="front" x_offset="${caster_offset_x}"/>
-  <!-- ==================== LiDAR ==================== -->
-  <link name="lidar_link">
-    <visual>
-      <geometry>
-        <cylinder radius="${lidar_radius}" length="${lidar_height}"/>
-      </geometry>
-      <origin xyz="0 0 0" rpy="0 0 0"/>
-      <material name="orange"/>
-    </visual>
-    <collision>
-      <geometry>
-        <cylinder radius="${lidar_radius}" length="${lidar_height}"/>
-      </geometry>
-      <origin xyz="0 0 0" rpy="0 0 0"/>
-    </collision>
-    <xacro:cylinder_inertia m="${lidar_mass}" r="${lidar_radius}" h="${lidar_height}"/>
-  </link>
-  <joint name="lidar_joint" type="fixed">
-    <parent link="base_link"/>
-    <child link="lidar_link"/>
-    <origin xyz="0 0 ${base_height/2 + lidar_offset_z}" rpy="0 0 0"/>
-  </joint>
-  <!-- LiDAR scan frame (센서 데이터 기준점) -->
-  <link name="laser_frame"/>
-  <joint name="laser_joint" type="fixed">
-    <parent link="lidar_link"/>
-    <child link="laser_frame"/>
-    <origin xyz="0 0 ${lidar_height/2}" rpy="0 0 0"/>
-  </joint>
-  <!-- ==================== IMU (Optional) ==================== -->
+  <!-- ==================== Casters (4 corners) ==================== -->
+  <xacro:caster prefix="front_left" x_reflect="1" y_reflect="1"/>
+  <xacro:caster prefix="front_right" x_reflect="1" y_reflect="-1"/>
+  <xacro:caster prefix="rear_left" x_reflect="-1" y_reflect="1"/>
+  <xacro:caster prefix="rear_right" x_reflect="-1" y_reflect="-1"/>
+  <!-- ==================== NanoScan3 LiDARs ==================== -->
+  <!-- Front-right LiDAR (1 o'clock position) -->
+  <xacro:nanoscan3 prefix="front"
+                   x="${lidar_front_x}"
+                   y="${lidar_front_y}"
+                   yaw="${lidar_front_yaw}"
+                   topic="scan_front"/>
+  <!-- Rear-left LiDAR (7 o'clock position) -->
+  <xacro:nanoscan3 prefix="rear"
+                   x="${lidar_rear_x}"
+                   y="${lidar_rear_y}"
+                   yaw="${lidar_rear_yaw}"
+                   topic="scan_rear"/>
+  <!-- ==================== IMU ==================== -->
   <link name="imu_link"/>
   <joint name="imu_joint" type="fixed">
